File: convector-booster-pcb/convector-booster-pcb.kicad_sch (KiCad schematic)
At the start: 2 parts

Commit message: Updated KiCad files.
Parts:
- removed R?: R, symbol Device:R
- added J1: Barrel_Jack, Connector_BarrelJack:BarrelJack_GCT_DCJ200-10-A_Horizontal, symbol Connector:Barrel_Jack
- added J2, J3, J4: Conn_01x03_Male, Connector_JST:JST_XH_B3B-XH-A_1x03_P2.50mm_Vertical, symbol Connector:Conn_01x03_Male
- added J5: Conn_01x04_Male, Connector_PinHeader_2.54mm:PinHeader_1x04_P2.54mm_Vertical, symbol Connector:Conn_01x04_Male
- added Q1: BSS138, Package_TO_SOT_SMD:SOT-23, symbol Transistor_FET:BSS138
- added R1, R2, R4: 10K, Resistor_SMD:R_1206_3216Metric_Pad1.30x1.75mm_HandSolder, symbol Device:R
- added R3, R5: 4K7, Resistor_SMD:R_1206_3216Metric_Pad1.30x1.75mm_HandSolder, symbol Device:R
- added R6: 27K4, Resistor_SMD:R_1206_3216Metric_Pad1.30x1.75mm_HandSolder, symbol Device:R
- added U1: L7805, Package_TO_SOT_THT:TO-220-3_Vertical, symbol Regulator_Linear:L7805
- gave numbers to parts that had none: 1
Connections:
- net GND: now reaches U2.10 (GND)
- net GND: now also J1.2, J2.1 (Pin_1), J3.1 (Pin_1), J4.1 (Pin_1), J5.1 (Pin_1), R4.1, R5.1, U1.2 (GND)
- net at U2.13 (SDA/D2): now also Q1.2 (S), R2.1
- net at U2.14 (SCL/D1): now also R4.2, R6.1
- net at U2.3 (D0): now also J2.2 (Pin_2), J3.2 (Pin_2), J4.2 (Pin_2), R3.1
- net +3V3: now reaches U2.8 (3V3)
- net +3V3: now also J2.3 (Pin_3), J3.3 (Pin_3), J4.3 (Pin_3), Q1.1 (G), R2.2, R3.2
- net +5V: now reaches U2.9 (5V)
- net +5V: now also U1.3 (OUT)
- new net: J5.3 (Pin_3), R5.2, R6.2
- new net: J5.4 (Pin_4), Q1.3 (D), R1.2
- new net +12V: J1.1, J5.2 (Pin_2), R1.1, U1.1 (IN)
Other:
- moved on the sheet: U2
